File: ProCo RAT Distorsion.kicad_pcb (KiCad board)
At the start: 2 copper layers, 68.6 x 76.2 mm, 53 parts, among them IC1 LM308

Commit message: correcciones y documentacion
Parts:
- C7: footprint prueba:C1 -> prueba:CP2
- D1: value (none) -> 1N4004
- D2, D3: value (none) -> D
- D4, D5: value (none) -> 1N4148
- D6: value (none) -> LED
- Q1, Q2: value (none) -> BF245
- R4: value 2M2 -> 2,2M
- X1, X13, X14, X15, X16, X2, X3: value (none) -> JD_CONN_01X01
- X10, X11, X12, X4, X5, X6, X7, X8, X9: value (none) -> JD_CONN_01X01; footprint prueba:Pad_2,5 -> prueba:PAD_OVAL
- moved C7 0.64 mm to (131.4, 118.1)
- turned X10 to 270 degrees
- turned X11 to 270 degrees
- turned X12 to 270 degrees
- turned X4 to 270 degrees
- turned X5 to 270 degrees
- turned X6 to 270 degrees
- turned X7 to 270 degrees
- turned X8 to 270 degrees
- turned X9 to 270 degrees
Routing:
- net Earth: track 277.4 -> 276.1 mm
