File: ProCo RAT Distorsion.sch (KiCad schematic (older format))
At the start: 60 parts, among them IC1 LM308, J1 Jack, J2 Jack_3.5, J3 Jack_3.5, Q1 Q_NJFET_GSD, Q2 Q_NJFET_GSD, X1 JD_CONN_01X01, X10 JD_CONN_01X01, X11 JD_CONN_01X01, X12 JD_CONN_01X01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

Commit message: correcciones y documentacion
Parts:
- added SW1A1, SW1B1: SW_DPDT_x2, symbol SW_DPDT_x2
- C7: footprint prueba:CP1 -> prueba:CP2
- J2: value Jack_3.5 -> in
- J3: value Jack_3.5 -> out
- POT1: value 100K -> 100K/LOG
- Q1, Q2: value Q_NJFET_GSD -> BF245
- X10, X11, X12, X4, X5, X6, X7, X8, X9: footprint prueba:Pad_2,5 -> prueba:PAD_OVAL
Connections:
- net at C3.1, R12.1, X2.1: now also SW1A1.1 (A); no longer J2.2 (T)
- net at POT3.2, X11.1, X3.1: now also SW1B1.2 (B); no longer J3.2 (T)
- net at Q2.1 (G), R13.2, X13.1: now also SW1B1.3 (C)
- new net: J3.2 (T), SW1A1.3 (C), SW1B1.1 (A)
- new net: J2.2 (T), SW1A1.2 (B)
Other:
- note added: "Esta línea es la que utiliza el original ya que el conmutador es sencillo"
- moved on the sheet: C13, D4, D5, D6, J2, J3, POT3, Q2, R11, R12, R13, R14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
